File: Boards/Headset board.sch (EAGLE design)
At the start: 4 parts

Commit message: PCB Boards
please review for my errors
Parts:
- added JP1: (no value), HyTechDevices:M04
- added JP2: (no value), HyTechDevices:M09
Connections:
- net N$1 renamed 9V
- net N$3 renamed 5V
- removed net N$2: G1.-, U$1.GND@3, U$2.GND, U$3.GND
- new net 3.3V: JP1.3, U$2.3.3V
- new net CSAG: JP2.3, U$2.D8(TX3)
- new net CSM: JP2.4, U$2.D7(RX3)
- new net GND: G1.-, JP1.4, U$1.GND@3, U$2.GND, U$3.GND
- new net SCL: JP1.1, U$2.D13
- new net SDA: JP1.2, U$2.D11
- new net SDD: JP2.1, JP2.2, U$2.D12
- new net SERIAL1: U$1.TX, U$2.D0(RX1)
- new net SERIAL2: U$1.RX, U$2.D1(TX1)
