File: Boards/camera board.brd (EAGLE design)
At the start: 60.9 x 84.8 mm, 6 parts

Commit message: PCB Boards
please review for my errors
Parts:
- added JP3, JP4: (no value), HyTechDevices:1X03
- JP2: device HyTechDevices:1X09 -> HyTechDevices:1X04
- moved JP1 17.7 mm to (50.8, 61.0), turned to 90 degrees
- moved JP2 17.7 mm to (50.8, 73.7), turned to 90 degrees
Connections:
- removed net CSAG: JP2.3, U$2.D8(TX3)
- removed net CSM: JP2.4, U$2.D7(RX3)
- removed net SCL: JP1.1, U$2.D13
- removed net SDA: JP1.2, U$2.D11
- removed net SDD: JP2.1, JP2.2, U$2.D12
- new net MOT1_1: JP1.2, U$2.D9(RX2)
- new net MOT1_2: JP1.1, U$2.D10(TX2)
- new net MOT2_1: JP2.2, U$2.D11
- new net MOT2_2: JP2.1, U$2.D12
- new net POT1: JP3.2, U$2.A6
- new net POT2: JP4.2, U$2.A9
- net 3.3V: now also JP3.1, JP4.1; no longer JP1.3
- net 9V: now also JP1.3, JP2.3
- net GND: now also JP2.4, JP3.3, JP4.3
- net SERIAL1: now also U$1.RX, U$2.D1(TX1); no longer U$1.TX, U$2.D0(RX1)
- net SERIAL2: now also U$1.TX, U$2.D0(RX1); no longer U$1.RX, U$2.D1(TX1)
Routing:
- net GND: track 159.0 -> 327.1 mm
- net SDA: track 100.8 -> 0.00 mm
- net MOT2_2: track 0.00 -> 85.0 mm
- net 9V: track 12.7 -> 94.1 mm
- net MOT2_1: track 0.00 -> 77.2 mm
- net CSAG: track 74.9 -> 0.00 mm
- net SCL: track 71.2 -> 0.00 mm
- net SDD: track 52.2 -> 0.00 mm
- net POT1: track 0.00 -> 51.6 mm
- net CSM: track 39.5 -> 0.00 mm
- net MOT1_1: track 0.00 -> 39.2 mm
- net MOT1_2: track 0.00 -> 38.8 mm
- net POT2: track 0.00 -> 24.3 mm
- net SERIAL2: track 42.2 -> 47.2 mm
- net SERIAL1: track 47.2 -> 42.2 mm
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
Commit message: New Board design
Parts:
- moved JP2 32.1 mm to (81.3, 63.5), turned to 270 degrees
- moved JP4 18.0 mm to (61.0, 66.0)
- moved JP3 7.62 mm to (61.0, 61.0)
- moved JP1 2.54 mm to (48.3, 61.0)
Connections:
- net POT2: now also U$2.A8; no longer U$2.A9
Routing:
- net 3.3V: track 52.1 -> 90.5 mm
- net 9V: track 94.1 -> 120.7 mm
- net GND: track 327.1 -> 348.2 mm
- net POT1: track 51.6 -> 32.3 mm
- net POT2: track 24.3 -> 41.9 mm
- net MOT2_1: track 77.2 -> 93.2 mm
- net MOT2_2: track 85.0 -> 96.0 mm
- net MOT1_2: track 38.8 -> 42.4 mm
- net MOT1_1: track 39.2 -> 42.6 mm
- net 5V: track 110.1 -> 108.8 mm
Other:
- board size 60.9 x 84.8 mm -> 60.9 x 69.5 mm
