File: Boards/Headset board.brd (EAGLE design)
At the start: 60.9 x 84.8 mm, 6 parts

Commit message: Board can't be printed
:(
Routing:
- net SDA: track 100.8 -> 99.6 mm
Other:
- board size 60.9 x 84.8 mm -> 58.4 x 84.8 mm
Changed lines of the file:
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@@
 <board>
 <plain>
-<wire x1="25.4" y1="0" x2="86.34" y2="0" width="0" layer="20"/>
-<wire x1="86.34" y1="0" x2="86.34" y2="84.76" width="0" layer="20"/>
-<wire x1="86.34" y1="84.76" x2="25.4" y2="84.76" width="0" layer="20"/>
+<wire x1="25.4" y1="0" x2="83.8" y2="0" width="0" layer="20"/>
+<wire x1="83.8" y1="0" x2="83.8" y2="84.76" width="0" layer="20"/>
+<wire x1="83.8" y1="84.76" x2="25.4" y2="84.76" width="0" layer="20"/>
 <wire x1="25.4" y1="84.76" x2="25.4" y2="0" width="0" layer="20"/>
 </plain>
@@
 <contactref element="JP1" pad="2"/>
 <wire x1="64.67740625" y1="19.0564" x2="60.96" y2="19.0564" width="0.4064" layer="16"/>
-<wire x1="60.96" y1="19.0564" x2="59.78259375" y2="19.0564" width="0.4064" layer="16"/>
 <wire x1="45.8690375" y1="53.3908" x2="31.7785125" y2="53.3908" width="0.4064" layer="16"/>
 <wire x1="46.8090375" y1="52.4508" x2="45.8690375" y2="53.3908" width="0.4064" layer="16"/>
@@
 <wire x1="30.0228" y1="55.1465125" x2="30.0228" y2="59.1534875" width="0.4064" layer="16"/>
 <wire x1="30.0228" y1="59.1534875" x2="31.7785125" y2="60.9092" width="0.4064" layer="16"/>
-<wire x1="56.1848" y1="50.67215625" x2="55.968478125" y2="50.888478125" width="0.4064" layer="16"/>
-<wire x1="55.968478125" y1="50.888478125" x2="54.40615625" y2="52.4508" width="0.4064" layer="16"/>
+<wire x1="57.4168" y1="49.44015625" x2="54.40615625" y2="52.4508" width="0.4064" layer="16"/>
 <wire x1="54.40615625" y1="52.4508" x2="46.8090375" y2="52.4508" width="0.4064" layer="16"/>
 <wire x1="31.7785125" y1="60.9092" x2="32.6869375" y2="60.9092" width="0.4064" layer="16"/>
@@
 <wire x1="65.4176" y1="20.84340625" x2="63.5" y2="22.76100625" width="0.4064" layer="16"/>
 <wire x1="60.96" y1="19.0564" x2="57.4168" y2="22.5996" width="0.4064" layer="16"/>
-<wire x1="57.4168" y1="49.44015625" x2="56.1848" y2="50.67215625" width="0.4064" layer="16"/>
 <wire x1="57.4168" y1="22.5996" x2="57.4168" y2="49.44015625" width="0.4064" layer="16"/>
 </signal>
